File: hardware/main_board.sch (EAGLE design)
At the start: 108 parts, among them IC1 IC_USBLC6-2, IC2 LM1117IMPX-3.3, IC3 STM32F107RCT, IC4 DP83848, IC5 LM1117MPX-2.5, U1 USD-SOCKETUSD, U2 VS1003, X2 CRYSTALS-NOGND-CFPX-217, X3 KUSBVX, Y1 CRYSTAL-GROUNDEDSMD-5X3.2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

Commit message: minor changes
Parts:
- removed SV1: (no value), con-harting-ml:ML14L
- added SV2: (no value), con-harting-ml:ML10L
Connections:
- new net PA10: IC3MCU.PA10, SV2.10
- new net PA8: IC3MCU.PA8, SV2.8
- new net PA9: IC3MCU.PA9, SV2.9
- new net PB14: IC3MCU.PB14, SV2.2
- new net PB15: IC3MCU.PB15, SV2.3
- new net PC6: IC3MCU.PC6, SV2.4
- new net PC7: IC3MCU.PC7, SV2.5
- new net PC8: IC3MCU.PC8, SV2.6
- new net PC9: IC3MCU.PC9, SV2.7
- net 3V: no longer SV1.1, SV1.2
- net GND: now also SV2.1; no longer SV1.3, SV1.4
Changed lines of the file:
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@@
 <part name="GND1" library="supply1" deviceset="GND" device=""/>
 <part name="GND18" library="supply1" deviceset="GND" device=""/>
-<part name="SV1" library="con-harting-ml" deviceset="ML14" device="L"/>
+<part name="SV2" library="con-harting-ml" deviceset="ML10" device="L"/>
 <part name="GND6" library="supply1" deviceset="GND" device=""/>
-<part name="GND10" library="supply1" deviceset="GND" device=""/>
 </parts>
 <sheets>
@@
 <instance part="GND1" gate="1" x="96.52" y="157.48"/>
 <instance part="GND18" gate="1" x="114.3" y="157.48"/>
-<instance part="SV1" gate="1" x="231.14" y="408.94"/>
-<instance part="GND6" gate="1" x="220.98" y="396.24"/>
-<instance part="GND10" gate="1" x="241.3" y="396.24"/>
+<instance part="SV2" gate="G$1" x="231.14" y="411.48"/>
+<instance part="GND6" gate="1" x="241.3" y="401.32"/>
 </instances>
 <busses>
@@
 </segment>
 <segment>
-<pinref part="SV1" gate="1" pin="4"/>
+<pinref part="SV2" gate="G$1" pin="1"/>
 <pinref part="GND6" gate="1" pin="GND"/>
-<wire x1="223.52" y1="403.86" x2="220.98" y2="403.86" width="0.1524" layer="91"/>
-<wire x1="220.98" y1="403.86" x2="220.98" y2="398.78" width="0.1524" layer="91"/>
-</segment>
-<segment>
-<pinref part="SV1" gate="1" pin="3"/>
-<pinref part="GND10" gate="1" pin="GND"/>
-<wire x1="238.76" y1="403.86" x2="241.3" y2="403.86" width="0.1524" layer="91"/>
-<wire x1="241.3" y1="403.86" x2="241.3" y2="398.78" width="0.1524" layer="91"/>
+<wire x1="238.76" y1="406.4" x2="241.3" y2="406.4" width="0.1524" layer="91"/>
+<wire x1="241.3" y1="406.4" x2="241.3" y2="403.86" width="0.1524" layer="91"/>
 </segment>
 </net>
@@
 <label x="223.52" y="449.58" size="1.4224" layer="95" rot="R180" xref="yes"/>
 </segment>
-<segment>
-<pinref part="SV1" gate="1" pin="2"/>
-<wire x1="223.52" y1="401.32" x2="215.9" y2="401.32" width="0.1524" layer="91"/>
-</segment>
-<segment>
-<pinref part="SV1" gate="1" pin="1"/>
-<wire x1="238.76" y1="401.32" x2="246.38" y2="401.32" width="0.1524" layer="91"/>
-</segment>
 </net>
 <net name="OSC32_IN" class="0">
@@
 </segment>
 </net>
+<net name="PB14" class="0">
+<segment>
+<pinref part="IC3" gate="MCU" pin="PB14"/>
+<wire x1="170.18" y1="243.84" x2="177.8" y2="243.84" width="0.1524" layer="91"/>
+</segment>
+<segment>
+<wire x1="223.52" y1="406.4" x2="215.9" y2="406.4" width="0.1524" layer="91"/>
+<pinref part="SV2" gate="G$1" pin="2"/>
+</segment>
+</net>
+<net name="PB15" class="0">
+<segment>
+<pinref part="IC3" gate="MCU" pin="PB15"/>
+<wire x1="170.18" y1="246.38" x2="177.8" y2="246.38" width="0.1524" layer="91"/>
+</segment>
+<segment>
+<wire x1="238.76" y1="408.94" x2="246.38" y2="408.94" width="0.1524" layer="91"/>
+<pinref part="SV2" gate="G$1" pin="3"/>
+</segment>
+</net>
+<net name="PC6" class="0">
+<segment>
+<pinref part="IC3" gate="MCU" pin="PC6"/>
+<wire x1="124.46" y1="223.52" x2="114.3" y2="223.52" width="0.1524" layer="91"/>
+</segment>
+<segment>
+<wire x1="223.52" y1="408.94" x2="215.9" y2="408.94" width="0.1524" layer="91"/>
+<pinref part="SV2" gate="G$1" pin="4"/>
+</segment>
+</net>
+<net name="PC7" class="0">
+<segment>
+<pinref part="IC3" gate="MCU" pin="PC7"/>
+<wire x1="124.46" y1="226.06" x2="114.3" y2="226.06" width="0.1524" layer="91"/>
+</segment>
+<segment>
+<wire x1="238.76" y1="411.48" x2="246.38" y2="411.48" width="0.1524" layer="91"/>
+<pinref part="SV2" gate="G$1" pin="5"/>
+</segment>
+</net>
+<net name="PC8" class="0">
+<segment>
+<pinref part="IC3" gate="MCU" pin="PC8"/>
+<wire x1="124.46" y1="228.6" x2="114.3" y2="228.6" width="0.1524" layer="91"/>
+</segment>
+<segment>
+<wire x1="223.52" y1="411.48" x2="215.9" y2="411.48" width="0.1524" layer="91"/>
+<pinref part="SV2" gate="G$1" pin="6"/>
+</segment>
+</net>
+<net name="PC9" class="0">
+<segment>
+<pinref part="IC3" gate="MCU" pin="PC9"/>
+<wire x1="124.46" y1="231.14" x2="114.3" y2="231.14" width="0.1524" layer="91"/>
+</segment>
+<segment>
+<wire x1="238.76" y1="414.02" x2="246.38" y2="414.02" width="0.1524" layer="91"/>
+<pinref part="SV2" gate="G$1" pin="7"/>
+</segment>
+</net>
+<net name="PA8" class="0">
+<segment>
+<pinref part="IC3" gate="MCU" pin="PA8"/>
+<wire x1="170.18" y1="185.42" x2="177.8" y2="185.42" width="0.1524" layer="91"/>
+</segment>
+<segment>
+<wire x1="223.52" y1="414.02" x2="215.9" y2="414.02" width="0.1524" layer="91"/>
+<pinref part="SV2" gate="G$1" pin="8"/>
+</segment>
+</net>
+<net name="PA10" class="0">
+<segment>
+<pinref part="IC3" gate="MCU" pin="PA10"/>
+<wire x1="170.18" y1="190.5" x2="177.8" y2="190.5" width="0.1524" layer="91"/>
+</segment>
+<segment>
+<wire x1="223.52" y1="416.56" x2="215.9" y2="416.56" width="0.1524" layer="91"/>
+<pinref part="SV2" gate="G$1" pin="10"/>
+</segment>
+</net>
+<net name="PA9" class="0">
+<segment>
+<pinref part="IC3" gate="MCU" pin="PA9"/>
+<wire x1="170.18" y1="187.96" x2="177.8" y2="187.96" width="0.1524" layer="91"/>
+</segment>
+<segment>
+<wire x1="238.76" y1="416.56" x2="246.38" y2="416.56" width="0.1524" layer="91"/>
+<pinref part="SV2" gate="G$1" pin="9"/>
+</segment>
+</net>

Commit message: Minor changes
Parts:
- added C6: (no value), rcl:C-EUC0603
- added JP3: (no value), pinhead:PINHD-1X2/90
- added R12: (no value), rcl:R-EU_R0603
Connections:
- net 3V: now also JP3.1, R12.2
- net GND: now also C6.2, JP3.2
- net NRST: now also C6.1, R12.1
Other:
- moved on the sheet: C1, C3, R9
Changed lines of the file:
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@@
 <part name="SV2" library="con-harting-ml" deviceset="ML10" device="L"/>
 <part name="GND6" library="supply1" deviceset="GND" device=""/>
+<part name="JP3" library="pinhead" deviceset="PINHD-1X2" device="/90"/>
+<part name="GND10" library="supply1" deviceset="GND" device=""/>
+<part name="R12" library="rcl" deviceset="R-EU_" device="R0603"/>
+<part name="C6" library="rcl" deviceset="C-EU" device="C0603"/>
+<part name="GND11" library="supply1" deviceset="GND" device=""/>
 </parts>
 <sheets>
@@
 <instance part="GND2" gate="1" x="304.8" y="320.04"/>
 <instance part="X3" gate="G$1" x="370.84" y="350.52"/>
-<instance part="C3" gate="G$1" x="106.68" y="167.64"/>
+<instance part="C3" gate="G$1" x="78.74" y="167.64"/>
 <instance part="C4" gate="G$1" x="15.24" y="548.64"/>
 <instance part="GND5" gate="1" x="15.24" y="538.48" rot="MR0"/>
@@
 <instance part="R43" gate="G$1" x="558.8" y="-17.78" rot="R90"/>
 <instance part="R1" gate="G$1" x="391.16" y="-63.5" rot="R270"/>
-<instance part="C1" gate="G$1" x="96.52" y="167.64"/>
+<instance part="C1" gate="G$1" x="68.58" y="167.64"/>
 <instance part="IC3" gate="MCU" x="147.32" y="205.74"/>
 <instance part="IC3" gate="PWR" x="53.34" y="210.82"/>
 <instance part="GND3" gate="1" x="55.88" y="182.88"/>
-<instance part="GND4" gate="1" x="106.68" y="157.48"/>
+<instance part="GND4" gate="1" x="78.74" y="157.48"/>
 <instance part="C2" gate="G$1" x="20.32" y="332.74"/>
 <instance part="C10" gate="G$1" x="12.7" y="332.74"/>
@@
 <instance part="Y1" gate="G$1" x="20.32" y="342.9" rot="R90"/>
 <instance part="GND17" gate="1" x="27.94" y="314.96"/>
-<instance part="R9" gate="G$1" x="88.9" y="175.26"/>
-<instance part="GND1" gate="1" x="96.52" y="157.48"/>
-<instance part="GND18" gate="1" x="114.3" y="157.48"/>
+<instance part="R9" gate="G$1" x="60.96" y="175.26"/>
+<instance part="GND1" gate="1" x="68.58" y="157.48"/>
+<instance part="GND18" gate="1" x="86.36" y="157.48"/>
 <instance part="SV2" gate="G$1" x="231.14" y="411.48"/>
 <instance part="GND6" gate="1" x="241.3" y="401.32"/>
+<instance part="JP3" gate="G$1" x="223.52" y="469.9" rot="MR0"/>
+<instance part="GND10" gate="1" x="231.14" y="462.28"/>
+<instance part="R12" gate="G$1" x="101.6" y="185.42" rot="R90"/>
+<instance part="C6" gate="G$1" x="101.6" y="160.02"/>
+<instance part="GND11" gate="1" x="101.6" y="149.86"/>
 </instances>
 <busses>
@@
 <pinref part="C3" gate="G$1" pin="2"/>
 <pinref part="GND4" gate="1" pin="GND"/>
-<wire x1="106.68" y1="160.02" x2="106.68" y2="162.56" width="0.1524" layer="91"/>
+<wire x1="78.74" y1="160.02" x2="78.74" y2="162.56" width="0.1524" layer="91"/>
 </segment>
 <segment>
@@
 <pinref part="C1" gate="G$1" pin="2"/>
 <pinref part="GND1" gate="1" pin="GND"/>
-<wire x1="96.52" y1="160.02" x2="96.52" y2="162.56" width="0.1524" layer="91"/>
+<wire x1="68.58" y1="160.02" x2="68.58" y2="162.56" width="0.1524" layer="91"/>
 </segment>
 <segment>
 <pinref part="IC3" gate="MCU" pin="VSSA"/>
 <pinref part="GND18" gate="1" pin="GND"/>
-<wire x1="124.46" y1="172.72" x2="114.3" y2="172.72" width="0.1524" layer="91"/>
-<wire x1="114.3" y1="172.72" x2="114.3" y2="165.1" width="0.1524" layer="91"/>
+<wire x1="124.46" y1="172.72" x2="86.36" y2="172.72" width="0.1524" layer="91"/>
+<wire x1="86.36" y1="172.72" x2="86.36" y2="165.1" width="0.1524" layer="91"/>
 <pinref part="IC3" gate="MCU" pin="BOOT0"/>
-<wire x1="114.3" y1="165.1" x2="114.3" y2="160.02" width="0.1524" layer="91"/>
-<wire x1="124.46" y1="165.1" x2="114.3" y2="165.1" width="0.1524" layer="91"/>
-<junction x="114.3" y="165.1"/>
+<wire x1="86.36" y1="165.1" x2="86.36" y2="160.02" width="0.1524" layer="91"/>
+<wire x1="124.46" y1="165.1" x2="86.36" y2="165.1" width="0.1524" layer="91"/>
+<junction x="86.36" y="165.1"/>
 </segment>
 <segment>
@@
 <wire x1="238.76" y1="406.4" x2="241.3" y2="406.4" width="0.1524" layer="91"/>
 <wire x1="241.3" y1="406.4" x2="241.3" y2="403.86" width="0.1524" layer="91"/>
+</segment>
+<segment>
+<pinref part="GND10" gate="1" pin="GND"/>
+<wire x1="231.14" y1="469.9" x2="231.14" y2="464.82" width="0.1524" layer="91"/>
+<pinref part="JP3" gate="G$1" pin="2"/>
+<wire x1="231.14" y1="469.9" x2="226.06" y2="469.9" width="0.1524" layer="91"/>
+</segment>
+<segment>
+<pinref part="C6" gate="G$1" pin="2"/>
+<pinref part="GND11" gate="1" pin="GND"/>
+<wire x1="101.6" y1="152.4" x2="101.6" y2="154.94" width="0.1524" layer="91"/>
 </segment>
 </net>
@@
 <segment>
 <pinref part="R9" gate="G$1" pin="1"/>
-<wire x1="83.82" y1="175.26" x2="78.74" y2="175.26" width="0.1524" layer="91"/>
-<label x="78.74" y="175.26" size="1.4224" layer="95" rot="R180" xref="yes"/>
+<wire x1="55.88" y1="175.26" x2="50.8" y2="175.26" width="0.1524" layer="91"/>
+<label x="50.8" y="175.26" size="1.4224" layer="95" rot="R180" xref="yes"/>
 </segment>
 <segment>
@@
 <wire x1="231.14" y1="449.58" x2="223.52" y2="449.58" width="0.1524" layer="91"/>
 <label x="223.52" y="449.58" size="1.4224" layer="95" rot="R180" xref="yes"/>
+</segment>
+<segment>
+<wire x1="231.14" y1="472.44" x2="231.14" y2="480.06" width="0.1524" layer="91"/>
+<label x="231.14" y="480.06" size="1.4224" layer="95" rot="R90" xref="yes"/>
+<pinref part="JP3" gate="G$1" pin="1"/>
+<wire x1="231.14" y1="472.44" x2="226.06" y2="472.44" width="0.1524" layer="91"/>
+</segment>
+<segment>
+<pinref part="R12" gate="G$1" pin="2"/>
+<wire x1="101.6" y1="190.5" x2="101.6" y2="195.58" width="0.1524" layer="91"/>
+<label x="101.6" y="195.58" size="1.4224" layer="95" rot="R90" xref="yes"/>
 </segment>
 </net>
@@
 <pinref part="IC3" gate="MCU" pin="VBAT"/>
 <pinref part="C3" gate="G$1" pin="1"/>
-<wire x1="124.46" y1="177.8" x2="106.68" y2="177.8" width="0.1524" layer="91"/>
-<wire x1="106.68" y1="177.8" x2="106.68" y2="170.18" width="0.1524" layer="91"/>
+<wire x1="124.46" y1="177.8" x2="78.74" y2="177.8" width="0.1524" layer="91"/>
+<wire x1="78.74" y1="177.8" x2="78.74" y2="170.18" width="0.1524" layer="91"/>
 </segment>
 </net>
@@
 <pinref part="R9" gate="G$1" pin="2"/>
 <pinref part="IC3" gate="MCU" pin="VDDA"/>
-<wire x1="93.98" y1="175.26" x2="96.52" y2="175.26" width="0.1524" layer="91"/>
+<wire x1="66.04" y1="175.26" x2="68.58" y2="175.26" width="0.1524" layer="91"/>
 <pinref part="C1" gate="G$1" pin="1"/>
-<wire x1="96.52" y1="175.26" x2="124.46" y2="175.26" width="0.1524" layer="91"/>
-<wire x1="96.52" y1="170.18" x2="96.52" y2="175.26" width="0.1524" layer="91"/>
-<junction x="96.52" y="175.26"/>
+<wire x1="68.58" y1="175.26" x2="124.46" y2="175.26" width="0.1524" layer="91"/>
+<wire x1="68.58" y1="170.18" x2="68.58" y2="175.26" width="0.1524" layer="91"/>
+<junction x="68.58" y="175.26"/>
 </segment>
 </net>
@@
 <segment>
 <pinref part="IC3" gate="MCU" pin="NRST"/>
-<wire x1="124.46" y1="167.64" x2="119.38" y2="167.64" width="0.1524" layer="91"/>
-</segment>
-<segment>
+<wire x1="124.46" y1="167.64" x2="101.6" y2="167.64" width="0.1524" layer="91"/>
+<pinref part="R12" gate="G$1" pin="1"/>
+<wire x1="101.6" y1="167.64" x2="96.52" y2="167.64" width="0.1524" layer="91"/>
+<wire x1="101.6" y1="180.34" x2="101.6" y2="167.64" width="0.1524" layer="91"/>
+<junction x="101.6" y="167.64"/>
+<pinref part="C6" gate="G$1" pin="1"/>
+<wire x1="101.6" y1="167.64" x2="101.6" y2="162.56" width="0.1524" layer="91"/>
+<label x="96.52" y="167.64" size="1.4224" layer="95" rot="R180" xref="yes"/>
+</segment>
+<segment>

Commit message: UART3 TX trace added
Connections:
- new net UART_TX: IC3MCU.PB10, SV2.1
- net GND: no longer SV2.1
Changed lines of the file:
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@@
 <part name="GND18" library="supply1" deviceset="GND" device=""/>
 <part name="SV2" library="con-harting-ml" deviceset="ML10" device="L"/>
-<part name="GND6" library="supply1" deviceset="GND" device=""/>
 <part name="JP3" library="pinhead" deviceset="PINHD-1X2" device="/90"/>
 <part name="GND10" library="supply1" deviceset="GND" device=""/>
@@
 <instance part="GND18" gate="1" x="86.36" y="157.48"/>
 <instance part="SV2" gate="G$1" x="231.14" y="411.48"/>
-<instance part="GND6" gate="1" x="241.3" y="401.32"/>
 <instance part="JP3" gate="G$1" x="223.52" y="469.9" rot="MR0"/>
 <instance part="GND10" gate="1" x="231.14" y="462.28"/>
@@
 <wire x1="231.14" y1="444.5" x2="223.52" y2="444.5" width="0.1524" layer="91"/>
 <label x="223.52" y="444.5" size="1.4224" layer="95" rot="R180" xref="yes"/>
-</segment>
-<segment>
-<pinref part="SV2" gate="G$1" pin="1"/>
-<pinref part="GND6" gate="1" pin="GND"/>
-<wire x1="238.76" y1="406.4" x2="241.3" y2="406.4" width="0.1524" layer="91"/>
-<wire x1="241.3" y1="406.4" x2="241.3" y2="403.86" width="0.1524" layer="91"/>
 </segment>
 <segment>
@@
 </segment>
 </net>
+<net name="UART_TX" class="0">
+<segment>
+<pinref part="IC3" gate="MCU" pin="PB10"/>
+<wire x1="170.18" y1="233.68" x2="177.8" y2="233.68" width="0.1524" layer="91"/>
+</segment>
+<segment>
+<pinref part="SV2" gate="G$1" pin="1"/>
+<wire x1="238.76" y1="406.4" x2="246.38" y2="406.4" width="0.1524" layer="91"/>
+</segment>
+</net>

Commit message: USB overcurrent protection added
Parts:
- removed C5: (no value), rcl:CPOL-EUSMCA
- added C8: (no value), rcl:C-EUC0402
- added R14: (no value), rcl:R-EU_R0603
- added U3: (no value), FaBo-Supply:STMPS2151STR
Connections:
- new net 5V: C12.+, C13.1, C52.+, C53.1, F1.2, IC2.IN, IC5.IN, U3.IN
- new net USB_EN: IC3MCU.PC0, R14.2, U3.EN
- new net USB_OVERCURRENT: IC3MCU.PA5, U3.FAULT
- net 3V: now also C8.1
- net GND: now also C8.2, R14.1, U3.GND; no longer C5.-
- net VBUS: now also U3.OUT; no longer C12.+, C13.1, C5.+, C52.+, C53.1, F1.2, IC2.IN, IC5.IN
Other:
- moved on the sheet: C11, C27, C38, C4, C7, IC1, X3
