File: hardware/main_board.sch (EAGLE design)
At the start: 113 parts, among them IC1 IC_USBLC6-2, IC2 LM1117IMPX-3.3, IC3 STM32F107RCT, IC4 DP83848, IC5 LM1117MPX-2.5, U1 USD-SOCKETUSD, U2 VS1003, X2 CRYSTALS-NOGND-CFPX-217, X3 KUSBVX, Y1 CRYSTAL-GROUNDEDSMD-5X3.2, Y3 CRYSTAL-GROUNDEDSMD-5X3.2

Commit message: Ethernet AVDD filtering
Parts:
- added L3: (no value), dp_devices:FERRITE-0805
Connections:
- new net A3V: C16.1, C17.1, C21.1, C55.1, C59.1, IC4.ANA33VDD, L3.2, R10.2, R2.2, R3.2, R4.2, R5.2, R7.2, RJ1.P4, RJ1.P5
- net 3V: now also L3.1; no longer C16.1, C17.1, C21.1, C55.1, C59.1, IC4.ANA33VDD, R10.2, R2.2, R3.2, R4.2, R5.2, R7.2, RJ1.P4, RJ1.P5
